Commit message: Add combined RViz simulation control

File: src/arachne_description/urdf/scout/scout_wheel_type1_vendor.xacro (robot description, xacro)
@@ -44,9 +44,10 @@
             </collision>
         </link>
-        <joint name="${wheel_prefix}_wheel" type="fixed">
+        <joint name="${wheel_prefix}_wheel" type="continuous">
             <parent link="base_link"/>
             <child link="${wheel_prefix}_wheel_link"/>
             <xacro:insert_block name="joint_pose"/>
             <axis xyz="0 -1 0" rpy="0 0 0" />
+            <limit effort="20.0" velocity="20.0"/>
         </joint>
     </xacro:macro>

File: src/arachne_description/urdf/scout/scout_wheel_type2_vendor.xacro (robot description, xacro)
@@ -44,9 +44,10 @@
             </collision>
         </link>
-        <joint name="${wheel_prefix}_wheel" type="fixed">
+        <joint name="${wheel_prefix}_wheel" type="continuous">
             <parent link="base_link"/>
             <child link="${wheel_prefix}_wheel_link"/>
             <xacro:insert_block name="joint_pose"/>
             <axis xyz="0 -1 0" rpy="0 0 0" />
+            <limit effort="20.0" velocity="20.0"/>
         </joint>
     </xacro:macro>
