Commit message: Add high-level sequence executor

File: src/arachne_moveit_config/config/arachne_ag95.srdf.xacro (robot description, xacro)
@@ -36,4 +36,12 @@
     <joint name="aubo_wrist3_joint" value="0.0"/>
   </group_state>
+  <group_state name="grasp" group="aubo_arm">
+    <joint name="aubo_shoulder_joint" value="1.32"/>
+    <joint name="aubo_upperArm_joint" value="-0.78"/>
+    <joint name="aubo_foreArm_joint" value="-0.72"/>
+    <joint name="aubo_wrist1_joint" value="0.35"/>
+    <joint name="aubo_wrist2_joint" value="-1.32"/>
+    <joint name="aubo_wrist3_joint" value="0.0"/>
+  </group_state>
   <group_state name="lift" group="aubo_arm">
     <joint name="aubo_shoulder_joint" value="1.60"/>

File: src/arachne_moveit_config/config/arachne_ms42dc.srdf.xacro (robot description, xacro)
@@ -32,4 +32,12 @@
     <joint name="aubo_wrist3_joint" value="0.0"/>
   </group_state>
+  <group_state name="grasp" group="aubo_arm">
+    <joint name="aubo_shoulder_joint" value="1.32"/>
+    <joint name="aubo_upperArm_joint" value="-0.78"/>
+    <joint name="aubo_foreArm_joint" value="-0.72"/>
+    <joint name="aubo_wrist1_joint" value="0.35"/>
+    <joint name="aubo_wrist2_joint" value="-1.32"/>
+    <joint name="aubo_wrist3_joint" value="0.0"/>
+  </group_state>
   <group_state name="lift" group="aubo_arm">
     <joint name="aubo_shoulder_joint" value="1.60"/>
