Commit message: Add deterministic Aubo hardware scripts

File: src/arachne_description/urdf/gazebo/arachne_gazebo_plugins.xacro (robot description, xacro)
@@ -1,10 +1,10 @@
 <?xml version="1.0"?>
 <robot xmlns:xacro="http://www.ros.org/wiki/xacro">
-  <xacro:property name="demo_aubo_shoulder" value="1.664"/>
-  <xacro:property name="demo_aubo_upperArm" value="0.034"/>
-  <xacro:property name="demo_aubo_foreArm" value="-1.324"/>
-  <xacro:property name="demo_aubo_wrist1" value="0.034"/>
-  <xacro:property name="demo_aubo_wrist2" value="-1.732"/>
-  <xacro:property name="demo_aubo_wrist3" value="0.0"/>
+  <xacro:property name="demo_aubo_shoulder" value="-1.5407387550371199"/>
+  <xacro:property name="demo_aubo_upperArm" value="0.05937252214606485"/>
+  <xacro:property name="demo_aubo_foreArm" value="2.0350620214427786"/>
+  <xacro:property name="demo_aubo_wrist1" value="1.9717090402766757"/>
+  <xacro:property name="demo_aubo_wrist2" value="1.5416031029821449"/>
+  <xacro:property name="demo_aubo_wrist3" value="-0.002335565908067907"/>
   <xacro:macro name="arachne_gazebo_surface" params="link mu1:=0.9 mu2:=0.9">
     <gazebo reference="${link}">

File: src/arachne_moveit_config/config/arachne_ag95.srdf.xacro (robot description, xacro)
@@ -13,10 +13,10 @@
   </group>
   <group_state name="home" group="aubo_arm">
-    <joint name="aubo_shoulder_joint" value="1.664"/>
-    <joint name="aubo_upperArm_joint" value="0.034"/>
-    <joint name="aubo_foreArm_joint" value="-1.324"/>
-    <joint name="aubo_wrist1_joint" value="0.034"/>
-    <joint name="aubo_wrist2_joint" value="-1.732"/>
-    <joint name="aubo_wrist3_joint" value="0.0"/>
+    <joint name="aubo_shoulder_joint" value="-1.5407387550371199"/>
+    <joint name="aubo_upperArm_joint" value="0.05937252214606485"/>
+    <joint name="aubo_foreArm_joint" value="2.0350620214427786"/>
+    <joint name="aubo_wrist1_joint" value="1.9717090402766757"/>
+    <joint name="aubo_wrist2_joint" value="1.5416031029821449"/>
+    <joint name="aubo_wrist3_joint" value="-0.002335565908067907"/>
   </group_state>
   <group_state name="ready" group="aubo_arm">

File: src/arachne_moveit_config/config/arachne_ms42dc.srdf.xacro (robot description, xacro)
@@ -9,10 +9,10 @@
   </group>
   <group_state name="home" group="aubo_arm">
-    <joint name="aubo_shoulder_joint" value="1.664"/>
-    <joint name="aubo_upperArm_joint" value="0.034"/>
-    <joint name="aubo_foreArm_joint" value="-1.324"/>
-    <joint name="aubo_wrist1_joint" value="0.034"/>
-    <joint name="aubo_wrist2_joint" value="-1.732"/>
-    <joint name="aubo_wrist3_joint" value="0.0"/>
+    <joint name="aubo_shoulder_joint" value="-1.5407387550371199"/>
+    <joint name="aubo_upperArm_joint" value="0.05937252214606485"/>
+    <joint name="aubo_foreArm_joint" value="2.0350620214427786"/>
+    <joint name="aubo_wrist1_joint" value="1.9717090402766757"/>
+    <joint name="aubo_wrist2_joint" value="1.5416031029821449"/>
+    <joint name="aubo_wrist3_joint" value="-0.002335565908067907"/>
   </group_state>
   <group_state name="ready" group="aubo_arm">
