Commit message: Add MS42DC gripper model

File: src/arachne_description/urdf/arachne.urdf.xacro (robot description, xacro)
@@ -13,5 +13,5 @@
   <xacro:include filename="aubo/aubo_i5_vendor.xacro"/>
   <xacro:include filename="aubo/aubo_i5_ros2_control.xacro"/>
-  <xacro:include filename="gripper/ag95.urdf.xacro"/>
+  <xacro:include filename="gripper/ms42dc.urdf.xacro"/>
   <xacro:include filename="mounts/scout_aubo_mount.xacro"/>
   <xacro:include filename="mounts/aubo_ms42dc_adapter.xacro"/>
@@ -22,10 +22,10 @@
   <xacro:arachne_aubo_i5_vendor parent="arm_mount_link"/>
   <xacro:arachne_aubo_ms42dc_adapter parent="tool0" xyz="$(arg tool_adapter_xyz)" rpy="$(arg tool_adapter_rpy)"/>
-  <xacro:arachne_ag95 parent="gripper_adapter_link"/>
+  <xacro:arachne_ms42dc parent="gripper_adapter_link"/>
   <xacro:if value="$(arg with_lidar)">
     <xacro:arachne_lidar parent="base_link"/>
   </xacro:if>
   <xacro:if value="$(arg with_ee_camera)">
-    <xacro:arachne_ee_camera parent="ag95_body"/>
+    <xacro:arachne_ee_camera parent="ms42dc_body_link"/>
   </xacro:if>
   <xacro:if value="$(arg with_ros2_control)">

File: src/arachne_description/urdf/gripper/ms42dc.urdf.xacro (robot description, xacro)
@@ -1,103 +1,31 @@
 <?xml version="1.0"?>
 <robot xmlns:xacro="http://www.ros.org/wiki/xacro">
-  <xacro:include filename="ms42dc_simple_collision.xacro"/>
   <xacro:macro name="arachne_ms42dc" params="prefix:='ms42dc_' parent">
-    <link name="${prefix}base_link">
+    <link name="${prefix}body_link">
       <visual>
-        <origin xyz="0 0 0.025" rpy="0 0 0"/>
+        <origin xyz="-0.049334103 0.049874070 0.016816675" rpy="1.570796327 0 0"/>
         <geometry>
-          <box size="0.11 0.08 0.05"/>
+          <mesh filename="package://arachne_description/meshes/gripper/ms42dc/MS42DC.stl" scale="0.001 0.001 0.001"/>
         </geometry>
         <material name="arachne_gripper"/>
       </visual>
       <collision>
-        <origin xyz="0 0 0.025" rpy="0 0 0"/>
+        <origin xyz="0 0 0.082318" rpy="0 0 0"/>
         <geometry>
-          <box size="0.11 0.08 0.05"/>
+          <box size="0.118 0.063 0.165"/>
         </geometry>
       </collision>
-      <xacro:box_inertial mass="0.6" x="0.11" y="0.08" z="0.05"/>
+      <xacro:box_inertial mass="0.6" x="0.118" y="0.063" z="0.165"/>
     </link>
     <joint name="${prefix}base_fixed_joint" type="fixed">
       <parent link="${parent}"/>
-      <child link="${prefix}base_link"/>
+      <child link="${prefix}body_link"/>
       <origin xyz="0 0 0" rpy="0 0 0"/>
     </joint>
-    <link name="${prefix}left_finger_base_link">
-      <xacro:ms42dc_finger_geometry material="arachne_gripper"/>
-      <xacro:box_inertial mass="0.08" x="0.022" y="0.026" z="0.11"/>
-    </link>
-    <link name="${prefix}right_finger_base_link">
-      <xacro:ms42dc_finger_geometry material="arachne_gripper"/>
-      <xacro:box_inertial mass="0.08" x="0.022" y="0.026" z="0.11"/>
-    </link>
-    <link name="${prefix}left_finger_tip_link">
-      <visual>
-        <origin xyz="0 0 0.025" rpy="0 0 0"/>
-        <geometry>
-          <box size="0.026 0.030 0.05"/>
-        </geometry>
-        <material name="arachne_dark"/>
-      </visual>
-      <collision>
-        <origin xyz="0 0 0.025" rpy="0 0 0"/>
-        <geometry>
-          <box size="0.026 0.030 0.05"/>
-        </geometry>
-      </collision>
-      <xacro:box_inertial mass="0.03" x="0.026" y="0.030" z="0.05"/>
-    </link>
-    <link name="${prefix}right_finger_tip_link">
-      <visual>
-        <origin xyz="0 0 0.025" rpy="0 0 0"/>
-        <geometry>
-          <box size="0.026 0.030 0.05"/>
-        </geometry>
-        <material name="arachne_dark"/>
-      </visual>
-      <collision>
-        <origin xyz="0 0 0.025" rpy="0 0 0"/>
-        <geometry>
-          <box size="0.026 0.030 0.05"/>
-        </geometry>
-      </collision>
-      <xacro:box_inertial mass="0.03" x="0.026" y="0.030" z="0.05"/>
-    </link>
-    <link name="${prefix}center_frame"/>
     <link name="grasp_frame"/>
-    <joint name="${prefix}left_finger_joint" type="prismatic">
-      <parent link="${prefix}base_link"/>
-      <child link="${prefix}left_finger_base_link"/>
-      <origin xyz="0 0.025 0.045" rpy="0 0 0"/>
-      <axis xyz="0 1 0"/>
-      <limit lower="0.0" upper="0.035" effort="30" velocity="0.04"/>
-    </joint>
-    <joint name="${prefix}right_finger_joint" type="prismatic">
-      <parent link="${prefix}base_link"/>
-      <child link="${prefix}right_finger_base_link"/>
-      <origin xyz="0 -0.025 0.045" rpy="0 0 0"/>
-      <axis xyz="0 -1 0"/>
-      <limit lower="0.0" upper="0.035" effort="30" velocity="0.04"/>
-      <mimic joint="${prefix}left_finger_joint" multiplier="1.0" offset="0.0"/>
-    </joint>
-    <joint name="${prefix}left_tip_joint" type="fixed">
-      <parent link="${prefix}left_finger_base_link"/>
-      <child link="${prefix}left_finger_tip_link"/>
-      <origin xyz="0 0 0.11" rpy="0 0 0"/>
-    </joint>
-    <joint name="${prefix}right_tip_joint" type="fixed">
-      <parent link="${prefix}right_finger_base_link"/>
-      <child link="${prefix}right_finger_tip_link"/>
-      <origin xyz="0 0 0.11" rpy="0 0 0"/>
-    </joint>
-    <joint name="${prefix}center_frame_joint" type="fixed">
-      <parent link="${prefix}base_link"/>
-      <child link="${prefix}center_frame"/>
-      <origin xyz="0 0 0.10" rpy="0 0 0"/>
-    </joint>
     <joint name="${prefix}grasp_frame_joint" type="fixed">
-      <parent link="${prefix}center_frame"/>
+      <parent link="${prefix}body_link"/>
       <child link="grasp_frame"/>
-      <origin xyz="0 0 0.085" rpy="0 0 0"/>
+      <origin xyz="0 0 0.165" rpy="0 0 0"/>
     </joint>
   </xacro:macro>

File: src/arachne_description/urdf/gripper/ms42dc_ros2_control.xacro (robot description, xacro)
@@ -2,14 +2,5 @@
 <robot xmlns:xacro="http://www.ros.org/wiki/xacro">
   <xacro:macro name="arachne_ms42dc_ros2_control" params="prefix:='ms42dc_'">
-    <ros2_control name="${prefix}gripper_system" type="system">
-      <hardware>
-        <plugin>mock_components/GenericSystem</plugin>
-      </hardware>
-      <joint name="${prefix}left_finger_joint">
-        <command_interface name="position"/>
-        <state_interface name="position"/>
-        <state_interface name="velocity"/>
-      </joint>
-    </ros2_control>
+    <!-- Control integration will be added after the MS42DC ROS examples and protocol are wrapped. -->
   </xacro:macro>
 </robot>

Commit message: Improve Gazebo Switch demo

File: src/arachne_description/urdf/arachne.urdf.xacro (robot description, xacro)
@@ -10,4 +10,6 @@
   <xacro:arg name="with_ros2_control" default="false"/>
   <xacro:arg name="with_gazebo_plugins" default="false"/>
+  <xacro:arg name="with_mimic_joints" default="true"/>
+  <xacro:arg name="gazebo_drive_wheels" default="false"/>
   <xacro:include filename="materials.xacro"/>
   <xacro:include filename="common_inertials.xacro"/>
@@ -21,10 +23,10 @@
   <xacro:include filename="sensors/ee_camera.xacro"/>
   <xacro:include filename="gazebo/arachne_gazebo_plugins.xacro"/>
-  <xacro:arachne_scout_2_vendor/>
+  <xacro:arachne_scout_2_vendor gazebo_drive_wheels="$(arg gazebo_drive_wheels)"/>
   <xacro:arachne_scout_aubo_mount parent="base_link" xyz="$(arg arm_mount_xyz)" rpy="$(arg arm_mount_rpy)"/>
   <xacro:arachne_aubo_i5_vendor parent="arm_mount_link"/>
   <xacro:arachne_aubo_ms42dc_adapter parent="tool0" xyz="$(arg tool_adapter_xyz)" rpy="$(arg tool_adapter_rpy)"/>
   <xacro:if value="${'$(arg gripper_type)' == 'ms42dc'}">
-    <xacro:arachne_ms42dc parent="gripper_adapter_link"/>
+    <xacro:arachne_ms42dc parent="gripper_adapter_link" mimic_right="$(arg with_mimic_joints)"/>
   </xacro:if>
   <xacro:if value="${'$(arg gripper_type)' == 'ag95'}">

File: src/arachne_description/urdf/gazebo/arachne_gazebo_plugins.xacro (robot description, xacro)
@@ -100,4 +100,24 @@
       <xacro:arachne_gazebo_surface link="ms42dc_left_finger_link" mu1="1.1" mu2="1.1"/>
       <xacro:arachne_gazebo_surface link="ms42dc_right_finger_link" mu1="1.1" mu2="1.1"/>
+      <gazebo>
+        <plugin filename="gz-sim-joint-position-controller-system" name="gz::sim::systems::JointPositionController">
+          <joint_name>ms42dc_left_finger_joint</joint_name>
+          <topic>/arachne/gazebo/ms42dc_left_finger/command</topic>
+          <p_gain>6.0</p_gain>
+          <i_gain>0.0</i_gain>
+          <d_gain>0.2</d_gain>
+          <cmd_max>2.0</cmd_max>
+          <cmd_min>-2.0</cmd_min>
+        </plugin>
+        <plugin filename="gz-sim-joint-position-controller-system" name="gz::sim::systems::JointPositionController">
+          <joint_name>ms42dc_right_finger_joint</joint_name>
+          <topic>/arachne/gazebo/ms42dc_right_finger/command</topic>
+          <p_gain>6.0</p_gain>
+          <i_gain>0.0</i_gain>
+          <d_gain>0.2</d_gain>
+          <cmd_max>2.0</cmd_max>
+          <cmd_min>-2.0</cmd_min>
+        </plugin>
+      </gazebo>
     </xacro:if>
   </xacro:macro>

File: src/arachne_description/urdf/gripper/ms42dc.urdf.xacro (robot description, xacro)
@@ -23,5 +23,5 @@
     </collision>
   </xacro:macro>
-  <xacro:macro name="arachne_ms42dc" params="prefix:='ms42dc_' parent">
+  <xacro:macro name="arachne_ms42dc" params="prefix:='ms42dc_' parent mimic_right:=true">
     <link name="${prefix}body_link"/>
     <joint name="${prefix}body_fixed_joint" type="fixed">
@@ -60,5 +60,7 @@
       <axis xyz="0 0 -1"/>
       <limit lower="-1.0" upper="0.0" effort="30.0" velocity="1.0"/>
-      <mimic joint="${prefix}left_finger_joint" multiplier="-1.0" offset="0.0"/>
+      <xacro:if value="${mimic_right}">
+        <mimic joint="${prefix}left_finger_joint" multiplier="-1.0" offset="0.0"/>
+      </xacro:if>
     </joint>
     <link name="${prefix}mid_link">

File: src/arachne_description/urdf/scout/scout_2_vendor.xacro (robot description, xacro)
@@ -2,5 +2,5 @@
 <robot xmlns:xacro="http://www.ros.org/wiki/xacro">
     <!-- Adapted from agilexrobotics/scout_ros2/scout_description/urdf/scout_v2.xacro. -->
-    <xacro:macro name="arachne_scout_2_vendor">
+    <xacro:macro name="arachne_scout_2_vendor" params="gazebo_drive_wheels:=false">
     <xacro:include filename="scout/scout_wheel_type1_vendor.xacro" />
     <xacro:include filename="scout/scout_wheel_type2_vendor.xacro" />
@@ -58,16 +58,32 @@
     <!-- wheel labeled from 0 to 3, conter-clockwise, starting from front right wheel -->
     <!-- motor 1 and 2 (left side) are mechanically installed in a reversed direction -->
-    <xacro:scout_wheel_type1 wheel_prefix="front_right">
-        <origin xyz="${wheelbase/2} ${-track/2} ${wheel_vertical_offset}" rpy="3.14 0 0" />
-    </xacro:scout_wheel_type1>
-    <xacro:scout_wheel_type2 wheel_prefix="front_left">
-        <origin xyz="${wheelbase/2} ${track/2} ${wheel_vertical_offset}" rpy="0 0 0" />
-    </xacro:scout_wheel_type2>
-    <xacro:scout_wheel_type1 wheel_prefix="rear_left">
-        <origin xyz="${-wheelbase/2} ${track/2} ${wheel_vertical_offset}" rpy="0 0 0" />
-    </xacro:scout_wheel_type1>
-    <xacro:scout_wheel_type2 wheel_prefix="rear_right">
-        <origin xyz="${-wheelbase/2} ${-track/2} ${wheel_vertical_offset}" rpy="3.14 0 0" />
-    </xacro:scout_wheel_type2>
+    <xacro:unless value="${gazebo_drive_wheels}">
+        <xacro:scout_wheel_type1 wheel_prefix="front_right">
+            <origin xyz="${wheelbase/2} ${-track/2} ${wheel_vertical_offset}" rpy="3.14 0 0" />
+        </xacro:scout_wheel_type1>
+        <xacro:scout_wheel_type2 wheel_prefix="front_left">
+            <origin xyz="${wheelbase/2} ${track/2} ${wheel_vertical_offset}" rpy="0 0 0" />
+        </xacro:scout_wheel_type2>
+        <xacro:scout_wheel_type1 wheel_prefix="rear_left">
+            <origin xyz="${-wheelbase/2} ${track/2} ${wheel_vertical_offset}" rpy="0 0 0" />
+        </xacro:scout_wheel_type1>
+        <xacro:scout_wheel_type2 wheel_prefix="rear_right">
+            <origin xyz="${-wheelbase/2} ${-track/2} ${wheel_vertical_offset}" rpy="3.14 0 0" />
+        </xacro:scout_wheel_type2>
+    </xacro:unless>
+    <xacro:if value="${gazebo_drive_wheels}">
+        <xacro:scout_wheel_type1 wheel_prefix="front_right" visual_rpy="3.14 0 0">
+            <origin xyz="${wheelbase/2} ${-track/2} ${wheel_vertical_offset}" rpy="0 0 0" />
+        </xacro:scout_wheel_type1>
+        <xacro:scout_wheel_type2 wheel_prefix="front_left">
+            <origin xyz="${wheelbase/2} ${track/2} ${wheel_vertical_offset}" rpy="0 0 0" />
+        </xacro:scout_wheel_type2>
+        <xacro:scout_wheel_type1 wheel_prefix="rear_left">
+            <origin xyz="${-wheelbase/2} ${track/2} ${wheel_vertical_offset}" rpy="0 0 0" />
+        </xacro:scout_wheel_type1>
+        <xacro:scout_wheel_type2 wheel_prefix="rear_right" visual_rpy="3.14 0 0">
+            <origin xyz="${-wheelbase/2} ${-track/2} ${wheel_vertical_offset}" rpy="0 0 0" />
+        </xacro:scout_wheel_type2>
+    </xacro:if>
     </xacro:macro>
 </robot>

File: src/arachne_description/urdf/scout/scout_wheel_type1_vendor.xacro (robot description, xacro)
@@ -24,5 +24,5 @@
 -->
 <robot xmlns:xacro="http://www.ros.org/wiki/xacro" name="scout_wheel">
-    <xacro:macro name="scout_wheel_type1" params="wheel_prefix *joint_pose">
+    <xacro:macro name="scout_wheel_type1" params="wheel_prefix visual_rpy:='0 0 0' *joint_pose">
         <link name="${wheel_prefix}_wheel_link">
             <inertial>
@@ -32,5 +32,5 @@
             </inertial>
             <visual>
-                <origin xyz="0 0 0" rpy="0 0 0" />
+                <origin xyz="0 0 0" rpy="${visual_rpy}" />
                 <geometry>
                     <mesh filename="package://scout_description/meshes/wheel_type1.dae" />

File: src/arachne_description/urdf/scout/scout_wheel_type2_vendor.xacro (robot description, xacro)
@@ -24,5 +24,5 @@
 -->
 <robot xmlns:xacro="http://www.ros.org/wiki/xacro" name="scout_wheel">
-    <xacro:macro name="scout_wheel_type2" params="wheel_prefix *joint_pose">
+    <xacro:macro name="scout_wheel_type2" params="wheel_prefix visual_rpy:='0 0 0' *joint_pose">
         <link name="${wheel_prefix}_wheel_link">
             <inertial>
@@ -32,5 +32,5 @@
             </inertial>
             <visual>
-                <origin xyz="0 0 0" rpy="0 0 0" />
+                <origin xyz="0 0 0" rpy="${visual_rpy}" />
                 <geometry>
                     <mesh filename="package://scout_description/meshes/wheel_type2.dae" />

Commit message: Add planning control scaffold

File: src/arachne_description/urdf/arachne.urdf.xacro (robot description, xacro)
@@ -15,7 +15,10 @@
   <xacro:include filename="common_inertials.xacro"/>
   <xacro:include filename="scout/scout_2_vendor.xacro"/>
+  <xacro:include filename="scout/scout_2_ros2_control.xacro"/>
   <xacro:include filename="aubo/aubo_i5_vendor.xacro"/>
   <xacro:include filename="aubo/aubo_i5_ros2_control.xacro"/>
   <xacro:include filename="gripper/ms42dc.urdf.xacro"/>
+  <xacro:include filename="gripper/ms42dc_ros2_control.xacro"/>
+  <xacro:include filename="gripper/ag95_ros2_control.xacro"/>
   <xacro:include filename="mounts/scout_aubo_mount.xacro"/>
   <xacro:include filename="mounts/aubo_ms42dc_adapter.xacro"/>
@@ -46,5 +49,12 @@
   </xacro:if>
   <xacro:if value="$(arg with_ros2_control)">
+    <xacro:arachne_scout_2_ros2_control/>
     <xacro:arachne_aubo_i5_ros2_control prefix="aubo_"/>
+    <xacro:if value="${'$(arg gripper_type)' == 'ms42dc'}">
+      <xacro:arachne_ms42dc_ros2_control prefix="ms42dc_"/>
+    </xacro:if>
+    <xacro:if value="${'$(arg gripper_type)' == 'ag95'}">
+      <xacro:arachne_ag95_ros2_control/>
+    </xacro:if>
   </xacro:if>
   <xacro:if value="$(arg with_gazebo_plugins)">

File: src/arachne_description/urdf/gripper/ms42dc_ros2_control.xacro (robot description, xacro)
@@ -2,5 +2,19 @@
 <robot xmlns:xacro="http://www.ros.org/wiki/xacro">
   <xacro:macro name="arachne_ms42dc_ros2_control" params="prefix:='ms42dc_'">
-    <!-- Control integration will be added after the MS42DC ROS examples and protocol are wrapped. -->
+    <ros2_control name="${prefix}gripper_system" type="system">
+      <hardware>
+        <plugin>mock_components/GenericSystem</plugin>
+      </hardware>
+      <joint name="${prefix}left_finger_joint">
+        <command_interface name="position"/>
+        <state_interface name="position"/>
+        <state_interface name="velocity"/>
+      </joint>
+      <joint name="${prefix}right_finger_joint">
+        <command_interface name="position"/>
+        <state_interface name="position"/>
+        <state_interface name="velocity"/>
+      </joint>
+    </ros2_control>
   </xacro:macro>
 </robot>

Commit message: Add sensor rack camera and C16 model

File: src/arachne_description/urdf/arachne.urdf.xacro (robot description, xacro)
@@ -7,5 +7,12 @@
   <xacro:arg name="gripper_type" default="ms42dc"/>
   <xacro:arg name="with_lidar" default="true"/>
-  <xacro:arg name="with_ee_camera" default="false"/>
+  <xacro:arg name="with_ee_camera" default="true"/>
+  <xacro:arg name="with_rear_rack" default="true"/>
+  <xacro:arg name="rear_rack_xyz" default="-0.16 0.0 0.105"/>
+  <xacro:arg name="rear_rack_rpy" default="0.0 0.0 1.57079632679"/>
+  <xacro:arg name="lidar_xyz" default="0.0 0.035 0.6223"/>
+  <xacro:arg name="lidar_rpy" default="0.0 0.0 0.0"/>
+  <xacro:arg name="ee_camera_xyz" default="0.0 0.0 0.0"/>
+  <xacro:arg name="ee_camera_rpy" default="0.0 0.0 0.0"/>
   <xacro:arg name="with_ros2_control" default="false"/>
   <xacro:arg name="with_gazebo_plugins" default="false"/>
@@ -23,4 +30,5 @@
   <xacro:include filename="mounts/scout_aubo_mount.xacro"/>
   <xacro:include filename="mounts/aubo_ms42dc_adapter.xacro"/>
+  <xacro:include filename="sensors/rear_rack.xacro"/>
   <xacro:include filename="sensors/lidar.xacro"/>
   <xacro:include filename="sensors/ee_camera.xacro"/>
@@ -37,14 +45,17 @@
     <xacro:arachne_ag95 parent="gripper_adapter_link"/>
   </xacro:if>
+  <xacro:if value="$(arg with_rear_rack)">
+    <xacro:arachne_rear_sensor_rack parent="base_link" xyz="$(arg rear_rack_xyz)" rpy="$(arg rear_rack_rpy)"/>
+  </xacro:if>
   <xacro:if value="$(arg with_lidar)">
-    <xacro:arachne_lidar parent="base_link"/>
+    <xacro:if value="$(arg with_rear_rack)">
+      <xacro:arachne_lidar parent="rear_rack_link" xyz="$(arg lidar_xyz)" rpy="$(arg lidar_rpy)"/>
+    </xacro:if>
+    <xacro:if value="${'$(arg with_rear_rack)' == 'false'}">
+      <xacro:arachne_lidar parent="base_link"/>
+    </xacro:if>
   </xacro:if>
   <xacro:if value="$(arg with_ee_camera)">
-    <xacro:if value="${'$(arg gripper_type)' == 'ms42dc'}">
-      <xacro:arachne_ee_camera parent="ms42dc_body_link"/>
-    </xacro:if>
-    <xacro:if value="${'$(arg gripper_type)' == 'ag95'}">
-      <xacro:arachne_ee_camera parent="ag95_body"/>
-    </xacro:if>
+    <xacro:arachne_ee_camera parent="gripper_adapter_link" xyz="$(arg ee_camera_xyz)" rpy="$(arg ee_camera_rpy)"/>
   </xacro:if>
   <xacro:if value="$(arg with_ros2_control)">

File: src/arachne_description/urdf/sensors/ee_camera.xacro (robot description, xacro)
@@ -1,25 +1,52 @@
 <?xml version="1.0"?>
 <robot xmlns:xacro="http://www.ros.org/wiki/xacro">
-  <xacro:macro name="arachne_ee_camera" params="parent xyz:='0.04 0 0.035' rpy:='0 0 0'">
+  <xacro:property name="ee_camera_support_scale" value="0.001"/>
+  <xacro:property name="ee_camera_support_visual_xyz" value="-0.031499998 -0.0815 -0.122628235"/>
+  <xacro:macro name="arachne_ee_camera" params="parent xyz:='0 0 0' rpy:='0 0 0' camera_xyz:='0.025 -0.069 0.03077' camera_rpy:='0 -1.57079632679 -1.57079632679'">
+    <link name="ee_camera_support_link">
+      <visual>
+        <origin xyz="${ee_camera_support_visual_xyz}" rpy="0 0 0"/>
+        <geometry>
+          <mesh filename="package://arachne_description/meshes/homemade/camera_support_colored.dae"/>
+        </geometry>
+        <material name="arachne_camera_support">
+          <color rgba="0.93 0.92 0.88 1.0"/>
+        </material>
+      </visual>
+      <collision>
+        <origin xyz="0 0.025 0.0025" rpy="0 0 0"/>
+        <geometry>
+          <box size="0.063 0.113 0.005"/>
+        </geometry>
+      </collision>
+      <xacro:box_inertial mass="0.04" x="0.063" y="0.113" z="0.005"/>
+    </link>
+    <joint name="ee_camera_support_joint" type="fixed">
+      <parent link="${parent}"/>
+      <child link="ee_camera_support_link"/>
+      <origin xyz="${xyz}" rpy="${rpy}"/>
+    </joint>
     <link name="ee_camera_link">
       <visual>
-        <origin xyz="0 0 0" rpy="0 0 0"/>
+        <origin xyz="-0.01587 -0.025 -0.0125" rpy="0 0 0"/>
         <geometry>
-          <box size="0.035 0.035 0.025"/>
+          <mesh filename="package://arachne_description/meshes/sensors/orbbec/gemini335_336/camera_link_colored.dae"/>
         </geometry>
-        <material name="arachne_sensor"/>
+        <material name="arachne_orbbec_camera">
+          <color rgba="0.015 0.016 0.018 1.0"/>
+        </material>
       </visual>
       <collision>
-        <origin xyz="0 0 0" rpy="0 0 0"/>
+        <origin xyz="0.0051 0 0.0125" rpy="0 0 0"/>
         <geometry>
-          <box size="0.035 0.035 0.025"/>
+          <box size="0.030 0.089 0.025"/>
         </geometry>
       </collision>
-      <xacro:box_inertial mass="0.08" x="0.035" y="0.035" z="0.025"/>
+      <xacro:box_inertial mass="0.08" x="0.030" y="0.089" z="0.025"/>
     </link>
     <joint name="ee_camera_joint" type="fixed">
-      <parent link="${parent}"/>
+      <parent link="ee_camera_support_link"/>
       <child link="ee_camera_link"/>
-      <origin xyz="${xyz}" rpy="${rpy}"/>
+      <origin xyz="${camera_xyz}" rpy="${camera_rpy}"/>
     </joint>
   </xacro:macro>

File: src/arachne_description/urdf/sensors/lidar.xacro (robot description, xacro)
@@ -4,17 +4,24 @@
     <link name="lidar_link">
       <visual>
-        <origin xyz="0 0 0.035" rpy="0 0 0"/>
+        <origin xyz="0 0 0.03895" rpy="0 0 0"/>
         <geometry>
-          <cylinder radius="0.055" length="0.07"/>
+          <cylinder radius="0.051" length="0.0779"/>
         </geometry>
         <material name="arachne_sensor"/>
       </visual>
+      <visual>
+        <origin xyz="0 0 0.085" rpy="0 0 0"/>
+        <geometry>
+          <cylinder radius="0.035" length="0.012"/>
+        </geometry>
+        <material name="arachne_dark"/>
+      </visual>
       <collision>
-        <origin xyz="0 0 0.035" rpy="0 0 0"/>
+        <origin xyz="0 0 0.03895" rpy="0 0 0"/>
         <geometry>
-          <cylinder radius="0.055" length="0.07"/>
+          <cylinder radius="0.051" length="0.0779"/>
         </geometry>
       </collision>
-      <xacro:cylinder_inertial mass="0.35" radius="0.055" length="0.07" axis="z"/>
+      <xacro:cylinder_inertial mass="0.8" radius="0.051" length="0.0779" axis="z"/>
     </link>
     <joint name="lidar_joint" type="fixed">
