Commit message: Add MoveIt grasp planning RViz demo

File: src/arachne_description/urdf/aubo/aubo_i5_vendor.xacro (robot description, xacro)
@@ -13,7 +13,5 @@
         <mesh filename="package://aubo_description/meshes/aubo_i5/visual/link0.DAE" />
       </geometry>
-      <material name="">
-        <color rgba="1 1 1 1" />
-      </material>
+      <material name="arachne_arm_joint_dark"/>
     </visual>
     <collision>
@@ -35,7 +33,5 @@
         <mesh filename="package://aubo_description/meshes/aubo_i5/visual/link1.DAE" />
       </geometry>
-      <material name="">
-        <color rgba="1 1 1 1" />
-      </material>
+      <material name="arachne_arm_shell"/>
     </visual>
     <collision>
@@ -64,7 +60,5 @@
         <mesh filename="package://aubo_description/meshes/aubo_i5/visual/link2.DAE" />
       </geometry>
-      <material name="">
-        <color rgba="1 1 1 1" />
-      </material>
+      <material name="arachne_arm_shell"/>
     </visual>
     <collision>
@@ -93,7 +87,5 @@
         <mesh filename="package://aubo_description/meshes/aubo_i5/visual/link3.DAE" />
       </geometry>
-      <material name="">
-        <color rgba="1 1 1 1" />
-      </material>
+      <material name="arachne_arm_joint_dark"/>
     </visual>
     <collision>
@@ -122,7 +114,5 @@
         <mesh filename="package://aubo_description/meshes/aubo_i5/visual/link4.DAE" />
       </geometry>
-      <material name="">
-        <color rgba="1 1 1 1" />
-      </material>
+      <material name="arachne_arm_shell"/>
     </visual>
     <collision>
@@ -151,7 +141,5 @@
         <mesh filename="package://aubo_description/meshes/aubo_i5/visual/link5.DAE" />
       </geometry>
-      <material name="">
-        <color rgba="1 1 1 1" />
-      </material>
+      <material name="arachne_arm_joint_dark"/>
     </visual>
     <collision>
@@ -180,7 +168,5 @@
         <mesh filename="package://aubo_description/meshes/aubo_i5/visual/link6.DAE" />
       </geometry>
-      <material name="">
-        <color rgba="1 1 1 1" />
-      </material>
+      <material name="arachne_arm_joint_dark"/>
     </visual>
     <collision>

File: src/arachne_description/urdf/materials.xacro (robot description, xacro)
@@ -10,4 +10,10 @@
     <color rgba="0.92 0.94 0.93 1.0"/>
   </material>
+  <material name="arachne_arm_shell">
+    <color rgba="0.88 0.90 0.86 1.0"/>
+  </material>
+  <material name="arachne_arm_joint_dark">
+    <color rgba="0.11 0.13 0.14 1.0"/>
+  </material>
   <material name="arachne_joint">
     <color rgba="0.18 0.22 0.24 1.0"/>

File: src/arachne_moveit_config/config/arachne_ag95.srdf.xacro (robot description, xacro)
@@ -70,4 +70,6 @@
   <end_effector name="ag95" parent_link="tool0" group="ag95_gripper" parent_group="aubo_arm"/>
   <disable_collisions link1="base_link" link2="arm_mount_link" reason="Adjacent"/>
+  <disable_collisions link1="base_link" link2="front_basket_link" reason="FixedAccessory"/>
+  <disable_collisions link1="base_link" link2="rear_rack_link" reason="FixedAccessory"/>
   <disable_collisions link1="arm_mount_link" link2="aubo_base_link" reason="Adjacent"/>
   <disable_collisions link1="arm_mount_link" link2="aubo_shoulder_Link" reason="Adjacent"/>

File: src/arachne_moveit_config/config/arachne_ms42dc.srdf.xacro (robot description, xacro)
@@ -58,4 +58,6 @@
   <end_effector name="ms42dc" parent_link="tool0" group="ms42dc_gripper" parent_group="aubo_arm"/>
   <disable_collisions link1="base_link" link2="arm_mount_link" reason="Adjacent"/>
+  <disable_collisions link1="base_link" link2="front_basket_link" reason="FixedAccessory"/>
+  <disable_collisions link1="base_link" link2="rear_rack_link" reason="FixedAccessory"/>
   <disable_collisions link1="arm_mount_link" link2="aubo_base_link" reason="Adjacent"/>
   <disable_collisions link1="arm_mount_link" link2="aubo_shoulder_Link" reason="Adjacent"/>
