Commit message: Fix robot model mounting and visualization

File: src/arachne_description/urdf/accessories/front_basket.xacro (robot description, xacro)
@@ -1,5 +1,5 @@
 <?xml version="1.0"?>
 <robot xmlns:xacro="http://www.ros.org/wiki/xacro">
-  <xacro:macro name="arachne_front_basket" params="parent xyz:='0.4655 0 -0.0735' rpy:='0 0 0'">
+  <xacro:macro name="arachne_front_basket" params="parent xyz:='0.4655 0 -0.0715' rpy:='0 0 0'">
     <link name="front_basket_link">
       <visual>

File: src/arachne_description/urdf/arachne.urdf.xacro (robot description, xacro)
@@ -1,8 +1,10 @@
 <?xml version="1.0"?>
 <robot name="arachne" xmlns:xacro="http://www.ros.org/wiki/xacro">
-  <xacro:arg name="arm_mount_xyz" default="0.22 0.0 0.155"/>
+  <xacro:arg name="arm_mount_xyz" default="0.22 0.0 0.105"/>
   <xacro:arg name="arm_mount_rpy" default="0.0 0.0 1.57079632679"/>
-  <xacro:arg name="tool_adapter_xyz" default="0.0 0.0 0.0"/>
-  <xacro:arg name="tool_adapter_rpy" default="0.0 0.0 0.785398163397"/>
+  <xacro:arg name="ee_support_xyz" default="0.0 0.0 0.0"/>
+  <xacro:arg name="ee_support_rpy" default="0.0 0.0 2.35619449019"/>
+  <xacro:arg name="tool_adapter_xyz" default="-0.049334103 0.049874070 0.021816675"/>
+  <xacro:arg name="tool_adapter_rpy" default="1.570796327 0.0 0.0"/>
   <xacro:arg name="gripper_type" default="ms42dc"/>
   <xacro:arg name="with_lidar" default="true"/>
@@ -10,12 +12,12 @@
   <xacro:arg name="with_rear_rack" default="true"/>
   <xacro:arg name="with_front_basket" default="true"/>
-  <xacro:arg name="front_basket_xyz" default="0.4655 0.0 -0.0735"/>
+  <xacro:arg name="front_basket_xyz" default="0.4655 0.0 -0.0715"/>
   <xacro:arg name="front_basket_rpy" default="0.0 0.0 0.0"/>
   <xacro:arg name="rear_rack_xyz" default="-0.16 0.0 0.105"/>
-  <xacro:arg name="rear_rack_rpy" default="0.0 0.0 0.0"/>
+  <xacro:arg name="rear_rack_rpy" default="0.0 0.0 1.57079632679"/>
   <xacro:arg name="lidar_xyz" default="0.0 0.035 0.6223"/>
   <xacro:arg name="lidar_rpy" default="0.0 0.0 0.0"/>
-  <xacro:arg name="ee_camera_xyz" default="0.0 0.0 0.0"/>
-  <xacro:arg name="ee_camera_rpy" default="0.0 0.0 0.0"/>
+  <xacro:arg name="ee_camera_xyz" default="0.0 -0.0741 0.005"/>
+  <xacro:arg name="ee_camera_rpy" default="0.0 0.0 1.57079632679"/>
   <xacro:arg name="with_ros2_control" default="false"/>
   <xacro:arg name="with_gazebo_plugins" default="false"/>
@@ -31,6 +33,4 @@
   <xacro:include filename="gripper/ms42dc_ros2_control.xacro"/>
   <xacro:include filename="gripper/ag95_ros2_control.xacro"/>
-  <xacro:include filename="mounts/scout_aubo_mount.xacro"/>
-  <xacro:include filename="mounts/aubo_ms42dc_adapter.xacro"/>
   <xacro:include filename="sensors/rear_rack.xacro"/>
   <xacro:include filename="sensors/lidar.xacro"/>
@@ -42,13 +42,12 @@
     <xacro:arachne_front_basket parent="base_link" xyz="$(arg front_basket_xyz)" rpy="$(arg front_basket_rpy)"/>
   </xacro:if>
-  <xacro:arachne_scout_aubo_mount parent="base_link" xyz="$(arg arm_mount_xyz)" rpy="$(arg arm_mount_rpy)"/>
-  <xacro:arachne_aubo_i5_vendor parent="arm_mount_link"/>
-  <xacro:arachne_aubo_ms42dc_adapter parent="tool0" xyz="$(arg tool_adapter_xyz)" rpy="$(arg tool_adapter_rpy)"/>
+  <xacro:arachne_aubo_i5_vendor parent="base_link" xyz="$(arg arm_mount_xyz)" rpy="$(arg arm_mount_rpy)"/>
+  <xacro:arachne_ee_camera_support parent="aubo_wrist3_Link" xyz="$(arg ee_support_xyz)" rpy="$(arg ee_support_rpy)"/>
   <xacro:if value="${'$(arg gripper_type)' == 'ms42dc'}">
-    <xacro:arachne_ms42dc parent="gripper_adapter_link" mimic_right="$(arg with_mimic_joints)"/>
+    <xacro:arachne_ms42dc parent="ee_camera_support_link" xyz="$(arg tool_adapter_xyz)" rpy="$(arg tool_adapter_rpy)" mimic_right="$(arg with_mimic_joints)"/>
   </xacro:if>
   <xacro:if value="${'$(arg gripper_type)' == 'ag95'}">
     <xacro:include filename="gripper/ag95.urdf.xacro"/>
-    <xacro:arachne_ag95 parent="gripper_adapter_link"/>
+    <xacro:arachne_ag95 parent="ee_camera_support_link" xyz="$(arg tool_adapter_xyz)" rpy="$(arg tool_adapter_rpy)"/>
   </xacro:if>
   <xacro:if value="$(arg with_rear_rack)">
@@ -64,5 +63,5 @@
   </xacro:if>
   <xacro:if value="$(arg with_ee_camera)">
-    <xacro:arachne_ee_camera parent="gripper_adapter_link" xyz="$(arg ee_camera_xyz)" rpy="$(arg ee_camera_rpy)"/>
+    <xacro:arachne_ee_camera_sensor parent="ee_camera_support_link" camera_xyz="$(arg ee_camera_xyz)" camera_rpy="$(arg ee_camera_rpy)"/>
   </xacro:if>
   <xacro:if value="$(arg with_ros2_control)">

File: src/arachne_description/urdf/aubo/aubo_i5_vendor.xacro (robot description, xacro)
@@ -1,5 +1,5 @@
 <robot xmlns:xacro="http://www.ros.org/wiki/xacro">
   <!-- Adapted from AuboRobot/aubo_description/urdf/aubo_i5.urdf. -->
-  <xacro:macro name="arachne_aubo_i5_vendor" params="parent">
+  <xacro:macro name="arachne_aubo_i5_vendor" params="parent xyz:='0 0 0' rpy:='0 0 0'">
   <link name="aubo_base_link">
     <inertial>
@@ -193,5 +193,5 @@
     <parent link="${parent}" />
     <child link="aubo_base_link" />
-    <origin xyz="0.0 0.0 0.0" rpy="0.0 0.0 0.0" />
+    <origin xyz="${xyz}" rpy="${rpy}" />
   </joint>
   </xacro:macro>

File: src/arachne_description/urdf/gripper/ag95.urdf.xacro (robot description, xacro)
@@ -2,7 +2,7 @@
 <robot xmlns:xacro="http://www.ros.org/wiki/xacro">
   <xacro:include filename="$(find dh_ag95_description)/urdf/dh_ag95_macro.xacro"/>
-  <xacro:macro name="arachne_ag95" params="parent">
+  <xacro:macro name="arachne_ag95" params="parent xyz:='0 0 0' rpy:='0 0 0'">
     <xacro:dh_ag95_gripper prefix="" parent="${parent}" grasp_link_offset="0.145">
-      <origin xyz="0 0 0" rpy="0 0 0"/>
+      <origin xyz="${xyz}" rpy="${rpy}"/>
     </xacro:dh_ag95_gripper>
     <link name="grasp_frame"/>

File: src/arachne_description/urdf/gripper/ms42dc.urdf.xacro (robot description, xacro)
@@ -4,4 +4,6 @@
   <xacro:property name="ms42dc_cad_xyz" value="-0.049334103 0.049874070 0.016816675"/>
   <xacro:property name="ms42dc_cad_rpy" value="1.570796327 0 0"/>
+  <xacro:property name="ms42dc_grasp_xyz_from_base" value="0.049334103 0.121875263 0.049874070"/>
+  <xacro:property name="ms42dc_grasp_rpy_from_base" value="-1.570796327 0 0"/>
   <xacro:property name="ms42dc_left_pivot_xyz" value="0.0133341030359 0.0576833250744 0.0610740704713"/>
   <xacro:property name="ms42dc_left_visual_xyz" value="-0.0133341030359 -0.0576833250744 -0.0610740704713"/>
@@ -25,11 +27,5 @@
     </collision>
   </xacro:macro>
-  <xacro:macro name="arachne_ms42dc" params="prefix:='ms42dc_' parent mimic_right:=true">
-    <link name="${prefix}body_link"/>
-    <joint name="${prefix}body_fixed_joint" type="fixed">
-      <parent link="${parent}"/>
-      <child link="${prefix}body_link"/>
-      <origin xyz="0 0 0" rpy="0 0 0"/>
-    </joint>
+  <xacro:macro name="arachne_ms42dc" params="prefix:='ms42dc_' parent xyz:='0 0 0' rpy:='0 0 0' mimic_right:=true">
     <link name="${prefix}base_link">
       <xacro:arachne_ms42dc_mesh name="ms42dc_base"/>
@@ -37,7 +33,7 @@
     </link>
     <joint name="${prefix}base_frame_joint" type="fixed">
-      <parent link="${prefix}body_link"/>
+      <parent link="${parent}"/>
       <child link="${prefix}base_link"/>
-      <origin xyz="${ms42dc_cad_xyz}" rpy="${ms42dc_cad_rpy}"/>
+      <origin xyz="${xyz}" rpy="${rpy}"/>
     </joint>
     <link name="${prefix}left_finger_link">
@@ -77,7 +73,7 @@
     <link name="grasp_frame"/>
     <joint name="${prefix}grasp_frame_joint" type="fixed">
-      <parent link="${prefix}body_link"/>
+      <parent link="${prefix}base_link"/>
       <child link="grasp_frame"/>
-      <origin xyz="0 0 ${ms42dc_closed_tip_z - ms42dc_grasp_tip_inset}" rpy="0 0 0"/>
+      <origin xyz="${ms42dc_grasp_xyz_from_base}" rpy="${ms42dc_grasp_rpy_from_base}"/>
     </joint>
   </xacro:macro>

File: src/arachne_description/urdf/sensors/ee_camera.xacro (robot description, xacro)
@@ -3,5 +3,5 @@
   <xacro:property name="ee_camera_support_scale" value="0.001"/>
   <xacro:property name="ee_camera_support_visual_xyz" value="-0.031499998 -0.0815 -0.122628235"/>
-  <xacro:macro name="arachne_ee_camera" params="parent xyz:='0 0 0' rpy:='0 0 0' camera_xyz:='0.025 -0.069 0.03077' camera_rpy:='0 -1.57079632679 -1.57079632679'">
+  <xacro:macro name="arachne_ee_camera_support" params="parent xyz:='0 0 0' rpy:='0 0 0'">
     <link name="ee_camera_support_link">
       <visual>
@@ -27,7 +27,9 @@
       <origin xyz="${xyz}" rpy="${rpy}"/>
     </joint>
+  </xacro:macro>
+  <xacro:macro name="arachne_ee_camera_sensor" params="parent camera_xyz:='0.0 -0.0741 0.005' camera_rpy:='0.0 0.0 1.57079632679'">
     <link name="ee_camera_link">
       <visual>
-        <origin xyz="-0.01587 -0.025 -0.0125" rpy="0 0 0"/>
+        <origin xyz="0 0 0" rpy="0 0 0"/>
         <geometry>
           <mesh filename="package://arachne_description/meshes/sensors/orbbec/gemini335_336/camera_link_colored.dae"/>
@@ -46,8 +48,12 @@
     </link>
     <joint name="ee_camera_joint" type="fixed">
-      <parent link="ee_camera_support_link"/>
+      <parent link="${parent}"/>
       <child link="ee_camera_link"/>
       <origin xyz="${camera_xyz}" rpy="${camera_rpy}"/>
     </joint>
   </xacro:macro>
+  <xacro:macro name="arachne_ee_camera" params="parent xyz:='0 0 0' rpy:='0 0 0' camera_xyz:='0.0 -0.0741 0.005' camera_rpy:='0.0 0.0 1.57079632679'">
+    <xacro:arachne_ee_camera_support parent="${parent}" xyz="${xyz}" rpy="${rpy}"/>
+    <xacro:arachne_ee_camera_sensor parent="ee_camera_support_link" camera_xyz="${camera_xyz}" camera_rpy="${camera_rpy}"/>
+  </xacro:macro>
 </robot>

File: src/arachne_moveit_config/config/arachne_ag95.srdf.xacro (robot description, xacro)
@@ -68,10 +68,8 @@
     <joint name="right_inner_knuckle_joint" value="0.93"/>
   </group_state>
-  <end_effector name="ag95" parent_link="tool0" group="ag95_gripper" parent_group="aubo_arm"/>
-  <disable_collisions link1="base_link" link2="arm_mount_link" reason="Adjacent"/>
+  <end_effector name="ag95" parent_link="aubo_wrist3_Link" group="ag95_gripper" parent_group="aubo_arm"/>
+  <disable_collisions link1="base_link" link2="aubo_base_link" reason="Adjacent"/>
   <disable_collisions link1="base_link" link2="front_basket_link" reason="FixedAccessory"/>
   <disable_collisions link1="base_link" link2="rear_rack_link" reason="FixedAccessory"/>
-  <disable_collisions link1="arm_mount_link" link2="aubo_base_link" reason="Adjacent"/>
-  <disable_collisions link1="arm_mount_link" link2="aubo_shoulder_Link" reason="Adjacent"/>
   <disable_collisions link1="aubo_base_link" link2="aubo_shoulder_Link" reason="Adjacent"/>
   <disable_collisions link1="aubo_shoulder_Link" link2="aubo_upperArm_Link" reason="Adjacent"/>
@@ -81,13 +79,10 @@
   <disable_collisions link1="aubo_wrist2_Link" link2="aubo_wrist3_Link" reason="Adjacent"/>
   <disable_collisions link1="aubo_wrist3_Link" link2="tool0" reason="Adjacent"/>
-  <disable_collisions link1="tool0" link2="gripper_adapter_link" reason="Adjacent"/>
-  <disable_collisions link1="aubo_wrist3_Link" link2="gripper_adapter_link" reason="Never"/>
-  <disable_collisions link1="aubo_wrist3_Link" link2="ee_camera_support_link" reason="Never"/>
+  <disable_collisions link1="aubo_wrist3_Link" link2="ee_camera_support_link" reason="Adjacent"/>
   <disable_collisions link1="aubo_wrist3_Link" link2="ee_camera_link" reason="Never"/>
   <disable_collisions link1="tool0" link2="ee_camera_support_link" reason="Never"/>
   <disable_collisions link1="tool0" link2="ee_camera_link" reason="Never"/>
-  <disable_collisions link1="gripper_adapter_link" link2="ee_camera_support_link" reason="Adjacent"/>
-  <disable_collisions link1="gripper_adapter_link" link2="ee_camera_link" reason="Never"/>
   <disable_collisions link1="ee_camera_support_link" link2="ee_camera_link" reason="Adjacent"/>
-  <disable_collisions link1="gripper_adapter_link" link2="ag95_body" reason="Adjacent"/>
+  <disable_collisions link1="ee_camera_support_link" link2="ag95_body" reason="Adjacent"/>
+  <disable_collisions link1="tool0" link2="ag95_body" reason="Never"/>
 </robot>

File: src/arachne_moveit_config/config/arachne_ms42dc.srdf.xacro (robot description, xacro)
@@ -56,10 +56,8 @@
     <joint name="ms42dc_right_finger_joint" value="-0.6"/>
   </group_state>
-  <end_effector name="ms42dc" parent_link="tool0" group="ms42dc_gripper" parent_group="aubo_arm"/>
-  <disable_collisions link1="base_link" link2="arm_mount_link" reason="Adjacent"/>
+  <end_effector name="ms42dc" parent_link="aubo_wrist3_Link" group="ms42dc_gripper" parent_group="aubo_arm"/>
+  <disable_collisions link1="base_link" link2="aubo_base_link" reason="Adjacent"/>
   <disable_collisions link1="base_link" link2="front_basket_link" reason="FixedAccessory"/>
   <disable_collisions link1="base_link" link2="rear_rack_link" reason="FixedAccessory"/>
-  <disable_collisions link1="arm_mount_link" link2="aubo_base_link" reason="Adjacent"/>
-  <disable_collisions link1="arm_mount_link" link2="aubo_shoulder_Link" reason="Adjacent"/>
   <disable_collisions link1="aubo_base_link" link2="aubo_shoulder_Link" reason="Adjacent"/>
   <disable_collisions link1="aubo_shoulder_Link" link2="aubo_upperArm_Link" reason="Adjacent"/>
@@ -69,39 +67,25 @@
   <disable_collisions link1="aubo_wrist2_Link" link2="aubo_wrist3_Link" reason="Adjacent"/>
   <disable_collisions link1="aubo_wrist3_Link" link2="tool0" reason="Adjacent"/>
-  <disable_collisions link1="tool0" link2="gripper_adapter_link" reason="Adjacent"/>
-  <disable_collisions link1="aubo_wrist3_Link" link2="gripper_adapter_link" reason="Never"/>
-  <disable_collisions link1="aubo_wrist3_Link" link2="ee_camera_support_link" reason="Never"/>
+  <disable_collisions link1="aubo_wrist3_Link" link2="ee_camera_support_link" reason="Adjacent"/>
   <disable_collisions link1="aubo_wrist3_Link" link2="ee_camera_link" reason="Never"/>
   <disable_collisions link1="tool0" link2="ee_camera_support_link" reason="Never"/>
   <disable_collisions link1="tool0" link2="ee_camera_link" reason="Never"/>
-  <disable_collisions link1="gripper_adapter_link" link2="ee_camera_support_link" reason="Adjacent"/>
-  <disable_collisions link1="gripper_adapter_link" link2="ee_camera_link" reason="Never"/>
   <disable_collisions link1="ee_camera_support_link" link2="ee_camera_link" reason="Adjacent"/>
-  <disable_collisions link1="gripper_adapter_link" link2="ms42dc_body_link" reason="Adjacent"/>
-  <disable_collisions link1="gripper_adapter_link" link2="ms42dc_base_link" reason="Never"/>
-  <disable_collisions link1="gripper_adapter_link" link2="ms42dc_mid_link" reason="Never"/>
-  <disable_collisions link1="gripper_adapter_link" link2="ms42dc_left_finger_link" reason="Never"/>
-  <disable_collisions link1="gripper_adapter_link" link2="ms42dc_right_finger_link" reason="Never"/>
-  <disable_collisions link1="ee_camera_support_link" link2="ms42dc_body_link" reason="Never"/>
-  <disable_collisions link1="ee_camera_support_link" link2="ms42dc_base_link" reason="Never"/>
+  <disable_collisions link1="ee_camera_support_link" link2="ms42dc_base_link" reason="Adjacent"/>
   <disable_collisions link1="ee_camera_support_link" link2="ms42dc_mid_link" reason="Never"/>
   <disable_collisions link1="ee_camera_support_link" link2="ms42dc_left_finger_link" reason="Never"/>
   <disable_collisions link1="ee_camera_support_link" link2="ms42dc_right_finger_link" reason="Never"/>
-  <disable_collisions link1="ee_camera_link" link2="ms42dc_body_link" reason="Never"/>
   <disable_collisions link1="ee_camera_link" link2="ms42dc_base_link" reason="Never"/>
   <disable_collisions link1="ee_camera_link" link2="ms42dc_mid_link" reason="Never"/>
   <disable_collisions link1="ee_camera_link" link2="ms42dc_left_finger_link" reason="Never"/>
   <disable_collisions link1="ee_camera_link" link2="ms42dc_right_finger_link" reason="Never"/>
-  <disable_collisions link1="aubo_wrist3_Link" link2="ms42dc_body_link" reason="Never"/>
   <disable_collisions link1="aubo_wrist3_Link" link2="ms42dc_base_link" reason="Never"/>
   <disable_collisions link1="aubo_wrist3_Link" link2="ms42dc_mid_link" reason="Never"/>
   <disable_collisions link1="aubo_wrist3_Link" link2="ms42dc_left_finger_link" reason="Never"/>
   <disable_collisions link1="aubo_wrist3_Link" link2="ms42dc_right_finger_link" reason="Never"/>
-  <disable_collisions link1="tool0" link2="ms42dc_body_link" reason="Never"/>
   <disable_collisions link1="tool0" link2="ms42dc_base_link" reason="Never"/>
   <disable_collisions link1="tool0" link2="ms42dc_mid_link" reason="Never"/>
   <disable_collisions link1="tool0" link2="ms42dc_left_finger_link" reason="Never"/>
   <disable_collisions link1="tool0" link2="ms42dc_right_finger_link" reason="Never"/>
-  <disable_collisions link1="ms42dc_body_link" link2="ms42dc_base_link" reason="Adjacent"/>
   <disable_collisions link1="ms42dc_base_link" link2="ms42dc_mid_link" reason="Adjacent"/>
   <disable_collisions link1="ms42dc_base_link" link2="ms42dc_left_finger_link" reason="Adjacent"/>
